File: Capstone_DataLogger/SD_Card_Reader.kicad_sch (KiCad schematic)
At the start: 4 parts, among them J2 MSD-4-A, U6 CD74HC4050E

Commit message: pcb connected except SD card
Parts:
- renumbered C3 to C1, C5 to C6, J2 to J4, U6 to U1
Changed lines of the file:
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@@
 	(wire
 		(pts
-			(xy 104.14 58.42) (xy 121.92 58.42)
+			(xy 101.6 58.42) (xy 121.92 58.42)
 		)
 		(stroke
@@
 	(hierarchical_label "MOSI"
 		(shape input)
-		(at 104.14 58.42 180)
+		(at 101.6 58.42 180)
 		(fields_autoplaced yes)
 		(effects
@@
 		(dnp no)
 		(fields_autoplaced yes)
-		(property "Reference" "U6"
+		(property "Reference" "U1"
 			(at 149.86 43.18 0)
 			(effects
@@
 		)
 		(instances
-			(project ""
-				(path "/3b56a84b-c06c-4c22-a01a-903db63bf091/58a600d6-fc19-4e0d-beb9-4eee34128a5c"
-					(reference "U6")
+			(project "Capstone_DataLogger"
+				(path "/3b56a84b-c06c-4c22-a01a-903db63bf091/9d44e97c-4d33-4cd2-a39b-04decca1d344"
+					(reference "U1")
 					(unit 1)
 				)
@@
 		(dnp no)
 		(fields_autoplaced yes)
-		(property "Reference" "#PWR016"
+		(property "Reference" "#PWR036"
 			(at 120.65 81.28 0)
 			(effects
@@
 		)
 		(instances
-			(project ""
-				(path "/3b56a84b-c06c-4c22-a01a-903db63bf091/58a600d6-fc19-4e0d-beb9-4eee34128a5c"
-					(reference "#PWR016")
+			(project "Capstone_DataLogger"
+				(path "/3b56a84b-c06c-4c22-a01a-903db63bf091/9d44e97c-4d33-4cd2-a39b-04decca1d344"
+					(reference "#PWR036")
 					(unit 1)
 				)
@@
 		(on_board yes)
 		(dnp no)
-		(property "Reference" "#PWR023"
+		(property "Reference" "#PWR029"
 			(at 109.22 102.87 0)
 			(effects
@@
 		(instances
 			(project "Capstone_DataLogger"
-				(path "/3b56a84b-c06c-4c22-a01a-903db63bf091/58a600d6-fc19-4e0d-beb9-4eee34128a5c"
-					(reference "#PWR023")
+				(path "/3b56a84b-c06c-4c22-a01a-903db63bf091/9d44e97c-4d33-4cd2-a39b-04decca1d344"
+					(reference "#PWR029")
 					(unit 1)
 				)
@@
 		(on_board yes)
 		(dnp no)
-		(property "Reference" "#PWR022"
+		(property "Reference" "#PWR037"
 			(at 123.19 97.79 0)
 			(effects
@@
 		(instances
 			(project "Capstone_DataLogger"
-				(path "/3b56a84b-c06c-4c22-a01a-903db63bf091/58a600d6-fc19-4e0d-beb9-4eee34128a5c"
-					(reference "#PWR022")
+				(path "/3b56a84b-c06c-4c22-a01a-903db63bf091/9d44e97c-4d33-4cd2-a39b-04decca1d344"
+					(reference "#PWR037")
 					(unit 1)
 				)
@@
 		(on_board yes)
 		(dnp no)
-		(property "Reference" "C3"
+		(property "Reference" "C1"
 			(at 111.76 38.0999 0)
 			(effects
@@
 		(instances
 			(project "Capstone_DataLogger"
-				(path "/3b56a84b-c06c-4c22-a01a-903db63bf091/58a600d6-fc19-4e0d-beb9-4eee34128a5c"
-					(reference "C3")
+				(path "/3b56a84b-c06c-4c22-a01a-903db63bf091/9d44e97c-4d33-4cd2-a39b-04decca1d344"
+					(reference "C1")
 					(unit 1)
 				)
@@
 		(dnp no)
 		(fields_autoplaced yes)
-		(property "Reference" "#PWR018"
+		(property "Reference" "#PWR048"
 			(at 180.34 80.01 0)
 			(effects
@@
 		)
 		(instances
-			(project ""
-				(path "/3b56a84b-c06c-4c22-a01a-903db63bf091/58a600d6-fc19-4e0d-beb9-4eee34128a5c"
-					(reference "#PWR018")
+			(project "Capstone_DataLogger"
+				(path "/3b56a84b-c06c-4c22-a01a-903db63bf091/9d44e97c-4d33-4cd2-a39b-04decca1d344"
+					(reference "#PWR048")
 					(unit 1)
 				)
@@
 		(dnp no)
 		(fields_autoplaced yes)
-		(property "Reference" "#PWR019"
+		(property "Reference" "#PWR030"
 			(at 115.57 50.8 0)
 			(effects
@@
 		(instances
 			(project "Capstone_DataLogger"
-				(path "/3b56a84b-c06c-4c22-a01a-903db63bf091/58a600d6-fc19-4e0d-beb9-4eee34128a5c"
-					(reference "#PWR019")
+				(path "/3b56a84b-c06c-4c22-a01a-903db63bf091/9d44e97c-4d33-4cd2-a39b-04decca1d344"
+					(reference "#PWR030")
 					(unit 1)
 				)
@@
 		(on_board yes)
 		(dnp no)
-		(property "Reference" "C5"
+		(property "Reference" "C6"
 			(at 116.84 92.71 90)
 			(effects
@@
 		(instances
 			(project "Capstone_DataLogger"
-				(path "/3b56a84b-c06c-4c22-a01a-903db63bf091/58a600d6-fc19-4e0d-beb9-4eee34128a5c"
-					(reference "C5")
+				(path "/3b56a84b-c06c-4c22-a01a-903db63bf091/9d44e97c-4d33-4cd2-a39b-04decca1d344"
+					(reference "C6")
 					(unit 1)
 				)
@@
 		(dnp no)
 		(fields_autoplaced yes)
-		(property "Reference" "#PWR06"
+		(property "Reference" "#PWR035"
 			(at 120.65 34.29 0)
 			(effects
@@
 		)
 		(instances
-			(project ""
-				(path "/3b56a84b-c06c-4c22-a01a-903db63bf091/58a600d6-fc19-4e0d-beb9-4eee34128a5c"
-					(reference "#PWR06")
+			(project "Capstone_DataLogger"
+				(path "/3b56a84b-c06c-4c22-a01a-903db63bf091/9d44e97c-4d33-4cd2-a39b-04decca1d344"
+					(reference "#PWR035")
 					(unit 1)
 				)
@@
 		(dnp no)
 		(fields_autoplaced yes)
-		(property "Reference" "J2"
+		(property "Reference" "J4"
 			(at 163.83 116.8399 0)
 			(effects
@@
 		)
 		(instances
-			(project ""
-				(path "/3b56a84b-c06c-4c22-a01a-903db63bf091/58a600d6-fc19-4e0d-beb9-4eee34128a5c"
-					(reference "J2")
+			(project "Capstone_DataLogger"
+				(path "/3b56a84b-c06c-4c22-a01a-903db63bf091/9d44e97c-4d33-4cd2-a39b-04decca1d344"
+					(reference "J4")
 					(unit 1)
 				)
@@
 		(on_board yes)
 		(dnp no)
-		(property "Reference" "#PWR021"
+		(property "Reference" "#PWR047"
 			(at 134.62 148.59 0)
 			(effects
@@
 		(instances
 			(project "Capstone_DataLogger"
-				(path "/3b56a84b-c06c-4c22-a01a-903db63bf091/58a600d6-fc19-4e0d-beb9-4eee34128a5c"
-					(reference "#PWR021")
+				(path "/3b56a84b-c06c-4c22-a01a-903db63bf091/9d44e97c-4d33-4cd2-a39b-04decca1d344"
+					(reference "#PWR047")
 					(unit 1)
 				)
