File: Capstone_DataLogger/Capstone_DataLogger.kicad_sch (KiCad schematic)
At the start: 0 parts

Commit message: Revised PCB
Parts:
- added J4, J5: S2B-PH-K-SLFSN, Capstone:CONN_S2B-PH-K-S_JST, symbol Capstone:S2B-PH-K-SLFSN
- added R5: 1k, Resistor_SMD:R_1206_3216Metric_Pad1.30x1.75mm_HandSolder, symbol Device:R
Connections:
- new net: J4.2, J5.1
- new net: J4.1, R5.2
- new net +5V: R5.1
- new net GND: J5.2

Commit message: Last revision before oreder
Parts:
- J4, J5: footprint Capstone:CONN_S2B-PH-K-S_JST -> Capstone:CONN_B2B-XH-A_JST
Other:
- sheet MCU ports: added THERM, VIBE_SENSE; removed none
- sheet Sensor_Interfacing ports: added AD0, THERM; removed none
Changed lines of the file:
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@@
+	(wire
+		(pts
+			(xy 177.8 86.36) (xy 170.18 86.36)
+		)
+		(stroke
+			(width 0)
+			(type default)
+		)
+	)
+	(wire
+		(pts
+			(xy 177.8 88.9) (xy 172.72 88.9)
+		)
+		(stroke
+			(width 0)
+			(type default)
+		)
+	)
 	(wire
 		(pts
@@
 	(wire
 		(pts
+			(xy 170.18 86.36) (xy 170.18 96.52)
+		)
+		(stroke
+			(width 0)
+			(type default)
+		)
+	)
+	(wire
+		(pts
 			(xy 149.86 88.9) (xy 162.56 88.9)
 		)
@@
 	(wire
 		(pts
+			(xy 170.18 96.52) (xy 149.86 96.52)
+		)
+		(stroke
+			(width 0)
+			(type default)
+		)
+	)
+	(wire
+		(pts
+			(xy 172.72 99.06) (xy 149.86 99.06)
+		)
+		(stroke
+			(width 0)
+			(type default)
+		)
+	)
+	(wire
+		(pts
 			(xy 167.64 93.98) (xy 167.64 83.82)
 		)
@@
 		(pts
 			(xy 149.86 91.44) (xy 165.1 91.44)
+		)
+		(stroke
+			(width 0)
+			(type default)
+		)
+	)
+	(wire
+		(pts
+			(xy 172.72 88.9) (xy 172.72 99.06)
 		)
 		(stroke
@@
 			)
 		)
-		(property "Footprint" "Capstone:CONN_S2B-PH-K-S_JST"
+		(property "Footprint" "Capstone:CONN_B2B-XH-A_JST"
 			(at 231.14 119.38 0)
 			(effects
@@
 			)
 		)
-		(property "Footprint" "Capstone:CONN_S2B-PH-K-S_JST"
+		(property "Footprint" "Capstone:CONN_B2B-XH-A_JST"
 			(at 231.14 97.79 0)
 			(effects
@@
 	(sheet
 		(at 177.8 78.74)
-		(size 25.4 7.62)
+		(size 25.4 13.97)
 		(fields_autoplaced yes)
 		(stroke
@@
 		)
 		(property "Sheetfile" "Sensor_interfacing.kicad_sch"
-			(at 177.8 86.9446 0)
+			(at 177.8 93.2946 0)
 			(effects
 				(font
@@
 		(pin "SCL" input
 			(at 177.8 81.28 180)
+			(effects
+				(font
+					(size 1.27 1.27)
+				)
+				(justify left)
+			)
+		)
+		(pin "AD0" input
+			(at 177.8 86.36 180)
+			(effects
+				(font
+					(size 1.27 1.27)
+				)
+				(justify left)
+			)
+		)
+		(pin "THERM" input
+			(at 177.8 88.9 180)
 			(effects
 				(font
@@
 			(effects
 				(font
+					(size 1.27 1.27)
+				)
+				(justify right)
+			)
+		)
+		(pin "VIBE_SENSE" input
+			(at 149.86 96.52 0)
+			(effects
+				(font
+					(size 1.27 1.27)
+				)
+				(justify right)
+			)
+		)
+		(pin "THERM" input
+			(at 149.86 99.06 0)
+			(effects
+				(font
