File: Capstone_DataLogger/Power_Interface.kicad_sch (KiCad schematic)
At the start: 3 parts, among them J3 S5B-PH-K-S, U5 TLV172IDCK

Commit message: Revised PCB
Parts:
- removed C4: 100p, Capacitor_SMD:C_1206_3216Metric_Pad1.33x1.80mm_HandSolder, symbol Device:C
- removed U5: TLV172IDCK, Package_TO_SOT_SMD:SOT-353_SC-70-5, symbol Amplifier_Operational:TLV172IDCK
Connections:
- net VBAT: now also J3.3

Commit message: Last revision before oreder
Parts:
- J3: footprint Capstone:CONN_S5B-PH-K-S_JST -> Capstone:CONN_B5B-XH-A_JST
Changed lines of the file:
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@@
 			)
 		)
-		(property "Footprint" "Capstone:CONN_S5B-PH-K-S_JST"
+		(property "Footprint" "Capstone:CONN_B5B-XH-A_JST"
 			(at 109.22 91.44 0)
 			(effects
