File: Capstone_DataLogger/Sensor_interfacing.kicad_sch (KiCad schematic)
At the start: 4 parts, among them J10 RJ9, J7 S4B-PH-K-SLFSN, J8 S4B-PH-K-SLFSN, J9 S4B-PH-K-SLFSN

Commit message: Revised PCB
Connections:
- net +5V_CTRL renamed +5V
Changed lines of the file:
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@@
 			)
 		)
-		(property "Value" "+5V_CTRL"
-			(at 142.24 125.73 0)
-			(effects
-				(font
-					(size 1.27 1.27)
-				)
+		(property "Value" "+5V"
+			(at 144.78 129.5399 0)
+			(effects
+				(font
+					(size 1.27 1.27)
+				)
+				(justify left)
 			)
 		)
@@
 			)
 		)
-		(property "Value" "+5V_CTRL"
-			(at 142.24 64.77 0)
-			(effects
-				(font
-					(size 1.27 1.27)
-				)
+		(property "Value" "+5V"
+			(at 144.78 68.5799 0)
+			(effects
+				(font
+					(size 1.27 1.27)
+				)
+				(justify left)
 			)
 		)
@@
 			)
 		)
-		(property "Value" "+5V_CTRL"
-			(at 142.24 31.75 0)
-			(effects
-				(font
-					(size 1.27 1.27)
-				)
+		(property "Value" "+5V"
+			(at 144.78 35.5599 0)
+			(effects
+				(font
+					(size 1.27 1.27)
+				)
+				(justify left)
 			)
 		)
@@
 			)
 		)
-		(property "Value" "+5V_CTRL"
-			(at 142.24 96.52 0)
-			(effects
-				(font
-					(size 1.27 1.27)
-				)
-			)
-		)
+		(property "Value" "+5V"
+			(at 144.78 100.3299 0)
+			(effects
+				(font
+					(size 1.27 1.27)
+				)
+				(justify left)
+			)
+		)

Commit message: Last revision before oreder
Parts:
- added J11: Conn_01x04_Socket, Connector_PinSocket_2.54mm:PinSocket_1x04_P2.54mm_Horizontal, symbol Connector:Conn_01x04_Socket
- added J12: S2B-PH-K-SLFSN, Capstone:CONN_B2B-XH-A_JST, symbol Capstone:S2B-PH-K-SLFSN
- added R7: 10k, Resistor_SMD:R_1206_3216Metric_Pad1.30x1.75mm_HandSolder, symbol Device:R
- J10: footprint Connector_RJ:RJ9_Evercom_5301-440xxx_Horizontal -> Capstone:RJ9
- J7, J8, J9: footprint Capstone:CONN_S4B-PH-K-S_JST -> Capstone:CONN_B4B-XH-A_JST
Connections:
- net +5V: now also J11.1 (Pin_1), J12.1
- net GND: now also J11.4 (Pin_4), R7.2
- new net AD0: J11.2 (Pin_2)
- new net THERM: J12.2, R7.1
- no-connect marks 0 -> 1
Other:
- note added: "P_SENSE"
- note added: "SENSOR_1"
- note added: "SENSOR_2"
- note added: "SENSOR_3"
- note added: "THERM"
- note added: "VIBE_SENSE"
- note removed: "Vibe Sens. Conn."
- moved on the sheet: J10, J7, J8, J9
