File: Capstone_DataLogger/RTC.kicad_sch (KiCad schematic)
At the start: 3 parts, among them U4 MCP7940M-I/P, Y2 32.768k

Commit message: Revised PCB
Parts:
- removed R1: 10k, Resistor_SMD:R_1206_3216Metric_Pad1.30x1.75mm_HandSolder, symbol Device:R
Connections:
- net at U4.1 (X1): now also Y2.1; no longer Y2.2
- net at U4.2 (X2): now also Y2.2; no longer Y2.1
- net MFP: no longer names the net of U4.7 (MFP)
- no-connect marks 0 -> 1
Changed lines of the file:
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@@
 		(comment 4 "Max Schatz")
 	)
-	(junction
+	(no_connect
 		(at 186.69 81.28)
-		(diameter 0)
-		(color 0 0 0 0)
-	)
-	(junction
-		(at 179.07 72.39)
-		(diameter 0)
-		(color 0 0 0 0)
 	)
 	(wire
@@
 	(wire
 		(pts
-			(xy 186.69 81.28) (xy 194.31 81.28)
-		)
-		(stroke
-			(width 0)
-			(type default)
-		)
-	)
-	(wire
-		(pts
 			(xy 172.72 86.36) (xy 194.31 86.36)
 		)
@@
 	(wire
 		(pts
-			(xy 186.69 80.01) (xy 186.69 81.28)
-		)
-		(stroke
-			(width 0)
-			(type default)
-		)
-	)
-	(wire
-		(pts
 			(xy 110.49 78.74) (xy 116.84 78.74)
 		)
@@
 	(wire
 		(pts
-			(xy 186.69 72.39) (xy 179.07 72.39)
+			(xy 97.79 85.09) (xy 110.49 85.09)
 		)
 		(stroke
@@
 	(wire
 		(pts
-			(xy 97.79 85.09) (xy 110.49 85.09)
-		)
-		(stroke
-			(width 0)
-			(type default)
-		)
-	)
-	(wire
-		(pts
-			(xy 97.79 76.2) (xy 97.79 74.93)
-		)
-		(stroke
-			(width 0)
-			(type default)
-		)
-	)
-	(wire
-		(pts
-			(xy 179.07 72.39) (xy 179.07 78.74)
-		)
-		(stroke
-			(width 0)
-			(type default)
-		)
-	)
-	(wire
-		(pts
-			(xy 179.07 69.85) (xy 179.07 72.39)
+			(xy 179.07 69.85) (xy 179.07 78.74)
 		)
 		(stroke
@@
 		(pts
 			(xy 97.79 74.93) (xy 110.49 74.93)
+		)
+		(stroke
+			(width 0)
+			(type default)
+		)
+	)
+	(wire
+		(pts
+			(xy 97.79 74.93) (xy 97.79 76.2)
 		)
 		(stroke
@@
 		(shape input)
 		(at 194.31 86.36 0)
-		(fields_autoplaced yes)
-		(effects
-			(font
-				(size 1.27 1.27)
-			)
-			(justify left)
-		)
-	)
-	(hierarchical_label "MFP"
-		(shape input)
-		(at 194.31 81.28 0)
 		(fields_autoplaced yes)
 		(effects
@@
 	)
 	(symbol
-		(lib_id "Device:R")
-		(at 186.69 76.2 0)
-		(unit 1)
-		(exclude_from_sim no)
-		(in_bom yes)
-		(on_board yes)
-		(dnp no)
-		(fields_autoplaced yes)
-		(property "Reference" "R1"
-			(at 189.23 74.9299 0)
-			(effects
-				(font
-					(size 1.27 1.27)
-				)
-				(justify left)
-			)
-		)
-		(property "Value" "10k"
-			(at 189.23 77.4699 0)
-			(effects
-				(font
-					(size 1.27 1.27)
-				)
-				(justify left)
-			)
-		)
-		(property "Footprint" "Resistor_SMD:R_1206_3216Metric_Pad1.30x1.75mm_HandSolder"
-			(at 184.912 76.2 90)
-			(effects
-				(font
-					(size 1.27 1.27)
-				)
-				(hide yes)
-			)
-		)
-		(property "Datasheet" "~"
-			(at 186.69 76.2 0)
-			(effects
-				(font
-					(size 1.27 1.27)
-				)
-				(hide yes)
-			)
-		)
-		(property "Description" "Resistor"
-			(at 186.69 76.2 0)
-			(effects
-				(font
-					(size 1.27 1.27)
-				)
-				(hide yes)
-			)
-		)
-		(pin "2"
-		)
-		(pin "1"
-		)
-		(instances
-			(project ""
-				(path "/3b56a84b-c06c-4c22-a01a-903db63bf091/0affded7-eae9-4d34-9de7-008cd2663c25"
-					(reference "R1")
-					(unit 1)
-				)
-			)
-		)
-	)
-	(symbol
 		(lib_id "Capstone:MCP7940M-I_P")
 		(at 116.84 78.74 0)
@@
 		(lib_id "Device:Crystal")
 		(at 97.79 80.01 90)
+		(mirror x)
 		(unit 1)
 		(exclude_from_sim no)
@@
 		(on_board yes)
 		(dnp no)
-		(fields_autoplaced yes)
 		(property "Reference" "Y2"
-			(at 101.6 78.7399 90)
+			(at 101.6 81.2801 90)
 			(effects
 				(font
@@
 		)
 		(property "Value" "32.768k"
-			(at 101.6 81.2799 90)
-			(effects
-				(font
+			(at 101.6 78.7401 90)
+			(effects
+				(font

Commit message: Hypothetical final revision of datalogger
Parts:
- added R6: 10k, Resistor_SMD:R_1206_3216Metric_Pad1.30x1.75mm_HandSolder, symbol Device:R
Connections:
- net +5V: now also R6.1
- net MFP: now reaches U4.7 (MFP)
- net MFP: now also R6.2
- no-connect marks 1 -> 0
Changed lines of the file:
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@@
 		(comment 4 "Max Schatz")
 	)
-	(no_connect
-		(at 186.69 81.28)
+	(junction
+		(at 181.61 81.28)
+		(diameter 0)
+		(color 0 0 0 0)
+	)
+	(junction
+		(at 179.07 72.39)
+		(diameter 0)
+		(color 0 0 0 0)
 	)
 	(wire
@@
 	(wire
 		(pts
-			(xy 186.69 81.28) (xy 172.72 81.28)
+			(xy 181.61 81.28) (xy 194.31 81.28)
 		)
 		(stroke
@@
 	(wire
 		(pts
-			(xy 179.07 69.85) (xy 179.07 78.74)
+			(xy 181.61 81.28) (xy 172.72 81.28)
+		)
+		(stroke
+			(width 0)
+			(type default)
+		)
+	)
+	(wire
+		(pts
+			(xy 179.07 69.85) (xy 179.07 72.39)
 		)
 		(stroke
@@
 	(wire
 		(pts
+			(xy 179.07 72.39) (xy 179.07 78.74)
+		)
+		(stroke
+			(width 0)
+			(type default)
+		)
+	)
+	(wire
+		(pts
+			(xy 181.61 72.39) (xy 179.07 72.39)
+		)
+		(stroke
+			(width 0)
+			(type default)
+		)
+	)
+	(wire
+		(pts
 			(xy 97.79 74.93) (xy 110.49 74.93)
 		)
@@
 		(pts
 			(xy 97.79 74.93) (xy 97.79 76.2)
+		)
+		(stroke
+			(width 0)
+			(type default)
+		)
+	)
+	(wire
+		(pts
+			(xy 181.61 73.66) (xy 181.61 72.39)
 		)
 		(stroke
@@
 		(shape input)
 		(at 194.31 83.82 0)
+		(fields_autoplaced yes)
+		(effects
+			(font
+				(size 1.27 1.27)
+			)
+			(justify left)
+		)
+	)
+	(hierarchical_label "MFP"
+		(shape input)
+		(at 194.31 81.28 0)
 		(fields_autoplaced yes)
 		(effects
@@
 					(unit 1)
 				)
+			)
+		)
+	)
+	(symbol
+		(lib_id "Device:R")
+		(at 181.61 77.47 0)
+		(unit 1)
+		(exclude_from_sim no)
+		(in_bom yes)
+		(on_board yes)
+		(dnp no)
+		(fields_autoplaced yes)
+		(property "Reference" "R6"
+			(at 184.15 76.1999 0)
+			(effects
+				(font
+					(size 1.27 1.27)
+				)
+				(justify left)
+			)
+		)
+		(property "Value" "10k"
+			(at 184.15 78.7399 0)
+			(effects
+				(font
+					(size 1.27 1.27)
+				)
+				(justify left)
+			)
+		)
+		(property "Footprint" "Resistor_SMD:R_1206_3216Metric_Pad1.30x1.75mm_HandSolder"
+			(at 179.832 77.47 90)
+			(effects
+				(font
+					(size 1.27 1.27)
+				)
+				(hide yes)
+			)
+		)
+		(property "Datasheet" "~"
+			(at 181.61 77.47 0)
+			(effects
+				(font
+					(size 1.27 1.27)
+				)
+				(hide yes)
+			)
+		)
+		(property "Description" "Resistor"
+			(at 181.61 77.47 0)
+			(effects
+				(font
+					(size 1.27 1.27)
+				)
+				(hide yes)
+			)
+		)
+		(pin "1"
+		)
+		(pin "2"
+		)
+		(instances
+			(project ""
+				(path "/3b56a84b-c06c-4c22-a01a-903db63bf091/0affded7-eae9-4d34-9de7-008cd2663c25"
+					(reference "R6")
+					(unit 1)
+				)
