File: Capstone_DataLogger/Capstone_DataLogger.kicad_pcb (KiCad board)
At the start: 2 copper layers, 70 x 130 mm, 25 parts, among them J1 S2B-PH-K-SLFSN, J10 RJ9, J11 Conn_01x04_Socket, J12 S2B-PH-K-SLFSN, J2 S2B-PH-K-SLFSN, J3 S5B-PH-K-S, J4 S2B-PH-K-SLFSN, J5 S2B-PH-K-SLFSN, J6 Conn_01x08_Pin, J7 S4B-PH-K-SLFSN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

Commit message: Hypothetical final revision of datalogger
Parts:
- added R6: 10k, Resistor_SMD:R_1206_3216Metric_Pad1.30x1.75mm_HandSolder, F.Cu at (157.0, 62.5)
- added U5: IRLZ34NPBF, Capstone:TO-220AB_INF, F.Cu at (151.6, 101.5)
- U1: footprint Connector_Molex:Molex_Micro-Latch_53253-0970_1x09_P2.00mm_Vertical -> Connector_PinHeader_2.54mm:PinHeader_1x09_P2.54mm_Vertical
- moved U2 6.18 mm to (119.3, 75.0), turned to 180 degrees
- moved C2 3.91 mm to (147.5, 66.4)
- moved U3 3.75 mm to (136.7, 48.5)
- moved J6 2.02 mm to (154.0, 67.2)
- moved U1 0.30 mm to (169.5, 41.9), turned to 0 degrees
Connections:
- U2 pad J2-11: unconnected-(U2-IO27-PadJ2-11) -> /MCU/ESP_SLEEP
- U2 pad J2-2: /MCU/ESP_EN -> Net-(U2-EN)
- U3 pad 14: unconnected-(U3-PB0-Pad14) -> /MCU/ESP_SLEEP
- U3 pad 2: /MCU/ESP_RX -> /MCU/ESP_TX
- U3 pad 3: /MCU/ESP_TX -> /MCU/ESP_RX
- U3 pad 4: unconnected-(U3-PD2-Pad4) -> /MCU/MFP
- U4 pad 7: unconnected-(U4-MFP-Pad7) -> /MCU/MFP
Routing:
- net +3.3V: track 95.1 -> 174.4 mm
- net Net-(U2-EN): track 0.00 -> 64.7 mm
- net /MCU/MFP: track 0.00 -> 61.2 mm
- net /MCU/CMD: track 143.9 -> 92.3 mm
- net /MCU/CLK: track 107.9 -> 64.0 mm
- net /MCU/D3: track 117.7 -> 93.0 mm
- net /MCU/D1: track 85.9 -> 108.0 mm
- net /MCU/D2: track 128.9 -> 108.4 mm
- net +5V: track 61.2 -> 41.1 mm
- net /MCU/~{RESET}: track 42.1 -> 60.5 mm
- net /MCU/ESP_RX: track 31.8 -> 50.0 mm
- net /MCU/D0: track 72.9 -> 89.8 mm
- net /MCU/ESP_SLEEP: track 0.00 -> 14.1 mm
- net /MCU/ESP_TX: track 36.2 -> 45.1 mm
- net Net-(J1-Pad1): track 106.3 -> 98.3 mm, vias 1 -> 2
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Other:
- board text added: "+3V3"

Commit message: Last revision
Changed lines of the file:
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@@
 			(solder_mask_margin 0.102)
 		)
-		(model "C:/Users/mpsch/Downloads/ESP32_DEVKITC_32D/ESP32-DEVKITC-32D.step"
+		(model "${KIPRJMOD}/Capstone.pretty/ESP_Header_Asssembe v1.step"
 			(offset
-				(xyz 0 0 0)
+				(xyz 0 0 9.5)
 			)
 			(scale
@@
 			)
 			(rotate
-				(xyz -90 0 0)
+				(xyz 0 0 0)
 			)
 		)
@@
 	)
 	(gr_line
+		(start 165.608 64.516)
+		(end 172.466 64.516)
+		(stroke
+			(width 0.1)
+			(type default)
+		)
+		(layer "F.SilkS")
+	)
+	(gr_line
+		(start 172.593 39.624)
+		(end 165.608 39.624)
+		(stroke
+			(width 0.1)
+			(type default)
+		)
+		(layer "F.SilkS")
+	)
+	(gr_line
 		(start 159.5 55.38)
 		(end 165.608 55.38)
 		(stroke
 			(width 0.1)
+			(type default)
+		)
+		(layer "F.SilkS")
+	)
+	(gr_line
+		(start 165.608 39.624)
+		(end 165.608 64.516)
+		(stroke
+			(width 0.1)
