File: PDU/Converters.kicad_sch (KiCad schematic)
At the start: 28 parts, among them J8 Conn_01x02_Socket, J9 Conn_01x02_Socket, U1 TPS564257DRLR, U9 TPS564257DRLR

Commit message: Last revision
Parts:
- removed J8, J9: Conn_01x02_Socket, Connector_PinHeader_2.54mm:PinHeader_1x02_P2.54mm_Vertical, symbol Connector:Conn_01x02_Socket
- added C28, C9: 22u, Capacitor_SMD:C_1206_3216Metric_Pad1.33x1.80mm_HandSolder, symbol Device:C
- added C29, C7: 100n, Capacitor_SMD:C_1206_3216Metric_Pad1.33x1.80mm_HandSolder, symbol Device:C
- added C6: 10u, Capacitor_SMD:C_1206_3216Metric_Pad1.33x1.80mm_HandSolder, symbol Device:C
- added C8: 10p, Resistor_SMD:R_1206_3216Metric_Pad1.30x1.75mm_HandSolder, symbol Device:C
- added L4: 4.7u, Inductor_SMD:L_Bourns_SRP7028A_7.3x6.6mm, symbol Device:L
- added R34: 113k, Resistor_SMD:R_1206_3216Metric_Pad1.30x1.75mm_HandSolder, symbol Device:R
- added R35: 30k, Resistor_SMD:R_1206_3216Metric_Pad1.30x1.75mm_HandSolder, symbol Device:R
- added R36, R38: 10k, Resistor_SMD:R_1206_3216Metric_Pad1.30x1.75mm_HandSolder, symbol Device:R
- added R37: 75.2k, Resistor_SMD:R_1206_3216Metric_Pad1.30x1.75mm_HandSolder, symbol Device:R
- added U3: TPS564257DRLR, Capstone:TPS564242DRLR_TEX, symbol Capstone:TPS564257DRLR
- C19, C21, C25, C26: footprint Capacitor_SMD:C_0805_2012Metric_Pad1.18x1.45mm_HandSolder -> Capacitor_SMD:C_1206_3216Metric_Pad1.33x1.80mm_HandSolder
- R21: value 220k -> 75.2k
Connections:
- net GND: now also C28.2, C29.2, C6.2, C7.2, C9.2, R35.2, R38.1, U3.3 (GND)
- net VIN: now also C1.1, C2.1, C22.1, C23.1, R1.1, R23.1, U1.1 (VIN), U9.1 (VIN), C6.1, C7.1, R34.1, U3.1 (VIN)
- new net: R34.2, R35.1, U3.5 (EN)
- new net: C8.2, R37.1, R38.2, U3.6 (FB)
- new net: L4.1, U3.2 (SW)
- new net: R36.1, U3.4 (PG)
- new net 5V_HEATER: C28.1, C29.1, C8.1, C9.1, L4.2, R36.2, R37.2
Other:
- moved on the sheet: C1, C19, C2, C20, C21, C22, C23, C24, C25, C26, C27, C3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
