File: PDU/NiMH_Charger.kicad_sch (KiCad schematic)
At the start: 11 parts, among them U6 BQ25172DSGR

Commit message: Last revision
Parts:
- removed TH1: 10k, Resistor_THT:R_Axial_DIN0204_L3.6mm_D1.6mm_P1.90mm_Vertical, symbol Device:Thermistor_NTC
- added J6: S2B-PH-K-SLFSN, CONN_S2B-PH-K-S_JST, symbol Capstone_2:S2B-PH-K-SLFSN
Connections:
- net GND: now also J6.1
- net at U6.3 (TS): now also J6.2
Changed lines of the file:
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@@
+	(wire
+		(pts
+			(xy 83.82 97.79) (xy 83.82 120.65)
+		)
+		(stroke
+			(width 0)
+			(type default)
+		)
+	)
 	(wire
 		(pts
@@
 	(wire
 		(pts
+			(xy 83.82 123.19) (xy 81.28 123.19)
+		)
+		(stroke
+			(width 0)
+			(type default)
+		)
+	)
+	(wire
+		(pts
 			(xy 195.58 99.06) (xy 195.58 101.6)
 		)
@@
 	(wire
 		(pts
-			(xy 83.82 106.68) (xy 83.82 110.49)
+			(xy 83.82 123.19) (xy 83.82 132.08)
 		)
 		(stroke
@@
 	(wire
 		(pts
-			(xy 83.82 97.79) (xy 83.82 99.06)
-		)
-		(stroke
-			(width 0)
-			(type default)
-		)
-	)
-	(wire
-		(pts
 			(xy 186.69 100.33) (xy 186.69 105.41)
 		)
@@
 		(pts
 			(xy 93.98 125.73) (xy 93.98 128.27)
+		)
+		(stroke
+			(width 0)
+			(type default)
+		)
+	)
+	(wire
+		(pts
+			(xy 81.28 120.65) (xy 83.82 120.65)
 		)
 		(stroke
@@
 	)
 	(symbol
+		(lib_id "Capstone_2:S2B-PH-K-SLFSN")
+		(at 81.28 123.19 180)
+		(unit 1)
+		(exclude_from_sim no)
+		(in_bom yes)
+		(on_board yes)
+		(dnp no)
+		(fields_autoplaced yes)
+		(property "Reference" "J6"
+			(at 72.39 113.03 0)
+			(effects
+				(font
+					(size 1.524 1.524)
+				)
+			)
+		)
+		(property "Value" "S2B-PH-K-SLFSN"
+			(at 72.39 115.57 0)
+			(effects
+				(font
+					(size 1.524 1.524)
+				)
+			)
+		)
+		(property "Footprint" "CONN_S2B-PH-K-S_JST"
+			(at 81.28 123.19 0)
+			(effects
+				(font
+					(size 1.27 1.27)
+					(italic yes)
+				)
+				(hide yes)
+			)
+		)
+		(property "Datasheet" "S2B-PH-K-SLFSN"
+			(at 81.28 123.19 0)
+			(effects
+				(font
+					(size 1.27 1.27)
+					(italic yes)
+				)
+				(hide yes)
+			)
+		)
+		(property "Description" ""
+			(at 81.28 123.19 0)
+			(effects
+				(font
+					(size 1.27 1.27)
+				)
+				(hide yes)
+			)
+		)
+		(pin "2"
+		)
+		(pin "1"
+		)
+		(instances
+			(project "PDU"
+				(path "/365e279d-a26e-42dd-bfe1-7a86883567c0/e5eaccd1-c3e9-4d78-9abc-df7aff823afe"
+					(reference "J6")
+					(unit 1)
+				)
+			)
+		)
+	)
+	(symbol
 		(lib_id "Device:C")
 		(at 68.58 96.52 0)
@@
 	)
 	(symbol
-		(lib_id "Device:Thermistor_NTC")
-		(at 83.82 102.87 0)
-		(unit 1)
-		(exclude_from_sim no)
-		(in_bom yes)
-		(on_board yes)
-		(dnp no)
-		(fields_autoplaced yes)
-		(property "Reference" "TH1"
-			(at 86.36 101.9174 0)
-			(effects
-				(font
-					(size 1.27 1.27)
-				)
-				(justify left)
-			)
-		)
-		(property "Value" "10k"
-			(at 86.36 104.4574 0)
-			(effects
-				(font
-					(size 1.27 1.27)
-				)
-				(justify left)
-			)
-		)
-		(property "Footprint" "Resistor_THT:R_Axial_DIN0204_L3.6mm_D1.6mm_P1.90mm_Vertical"
-			(at 83.82 101.6 0)
-			(effects
-				(font
-					(size 1.27 1.27)
-				)
-				(hide yes)
-			)
-		)
-		(property "Datasheet" "~"
-			(at 83.82 101.6 0)
-			(effects
-				(font
-					(size 1.27 1.27)
-				)
-				(hide yes)
-			)
-		)
-		(property "Description" "Temperature dependent resistor, negative temperature coefficient"
-			(at 83.82 102.87 0)
-			(effects
-				(font
-					(size 1.27 1.27)
-				)
-				(hide yes)
-			)
-		)
-		(pin "1"
-		)
-		(pin "2"
-		)
-		(instances
-			(project "PDU"
-				(path "/365e279d-a26e-42dd-bfe1-7a86883567c0/e5eaccd1-c3e9-4d78-9abc-df7aff823afe"
-					(reference "TH1")
-					(unit 1)
-				)
-			)
-		)
-	)
-	(symbol
 		(lib_id "power:GND")
 		(at 195.58 101.6 0)
@@
 	(symbol
 		(lib_id "power:GND")
-		(at 83.82 110.49 0)
+		(at 83.82 132.08 0)
 		(unit 1)
 		(exclude_from_sim no)
@@
 		(fields_autoplaced yes)
 		(property "Reference" "#PWR019"
-			(at 83.82 116.84 0)
+			(at 83.82 138.43 0)
 			(effects
 				(font
@@
 		)
 		(property "Value" "GND"
-			(at 83.82 115.57 0)
+			(at 83.82 137.16 0)
 			(effects
 				(font
@@
 		)
 		(property "Footprint" ""
-			(at 83.82 110.49 0)
+			(at 83.82 132.08 0)
 			(effects
 				(font
@@
 		)
 		(property "Datasheet" ""
-			(at 83.82 110.49 0)
+			(at 83.82 132.08 0)
 			(effects
 				(font
@@
 		)
 		(property "Description" "Power symbol creates a global label with name \"GND\" , ground"
-			(at 83.82 110.49 0)
-			(effects
-				(font
+			(at 83.82 132.08 0)
+			(effects
+				(font
