File: PDU/PDU.kicad_sch (KiCad schematic)
At the start: 12 parts, among them J10 Conn_01x02_Socket, J12 Conn_01x05_Pin, J2 USB_B_Micro, J6 Conn_01x02_Socket, J7 Conn_01x02_Socket, Q1 PMOS, Q2 NMOS, Q3 PMOS

Commit message: Last revision
Parts:
- removed J10, J6, J7: Conn_01x02_Socket, Connector_PinHeader_2.54mm:PinHeader_1x02_P2.54mm_Vertical, symbol Connector:Conn_01x02_Socket
- removed J12: Conn_01x05_Pin, Connector_PinHeader_2.54mm:PinHeader_1x05_P2.54mm_Vertical, symbol Connector:Conn_01x05_Pin
- removed Q1, Q3: PMOS, Package_TO_SOT_THT:TO-220-3_Horizontal_TabDown, symbol Simulation_SPICE:PMOS
- removed Q2: NMOS, Package_TO_SOT_THT:TO-220-3_Horizontal_TabDown, symbol Simulation_SPICE:NMOS
- removed R2, R4: 15, Capstone:res2_1-1625892-1_TEC, symbol Device:R
- added H1, H2: ReedSW MT, Capstone:ReedSW, symbol Mechanical:MountingHole
- added J1: S5B-PH-K-S, Capstone:CONN_B5B-XH-A_JST, symbol Capstone_2:S5B-PH-K-S
- added J3: 1935310, Capstone:CONN_1935310_PXC, symbol Capstone:1935310
- added J5: S2B-PH-K-SLFSN, CONN_S2B-PH-K-S_JST, symbol Capstone_2:S2B-PH-K-SLFSN
- added JP1: SolderJumper_2_Open, Jumper:SolderJumper-2_P1.3mm_Open_TrianglePad1.0x1.5mm, symbol Jumper:SolderJumper_2_Open
- added MOSFET1: DMP10H400SK3-13, Capstone:TO252-DPAK-DMP10H400SK3_DIO, symbol Capstone:DMP10H400SK3-13
- added Q3: IPD60R2K0PFD7SAUMA1, Capstone:DPAK229P994X240-3N, symbol Capstone:IPD60R2K0PFD7SAUMA1
- added R40: 100k, Resistor_SMD:R_1206_3216Metric_Pad1.30x1.75mm_HandSolder, symbol Device:R
- F1: footprint Capstone:FUS_LITTELFUSE_392_LTF -> Fuse:Fuse_2920_7451Metric_Pad2.10x5.45mm_HandSolder
- R3: value 10k -> 10; footprint Resistor_SMD:R_1206_3216Metric_Pad1.30x1.75mm_HandSolder -> Resistor_SMD:R_2512_6332Metric_Pad1.40x3.35mm_HandSolder
Connections:
- net +3.3V: now also J1.2
- net +5V: now also J1.1
- net Converters/VIN: now also MOSFET1.3 (S)
- net GND: now also J1.5, J3.2, Q3.3, R40.2
- net Ideal Diode/IN: now also JP1.2 (B), MOSFET1.1 (G), R40.1; no longer R3.1
- net NiMH Charger/OUT: now also R3.1, MOSFET1.2 (D); no longer F1.2
- net PWM_HEATER: now also J1.4, Q3.1
- net VBAT_SENSE: now also J1.3
- net VBAT_Monitor/VBAT_IN: now reaches R3.2
- net VBAT_Monitor/VBAT_IN: now also F1.2
- net MPPT/OUT renamed MPPT/+12V
- net MPPT/+12V: now also JP1.1 (A)
- new net: J5.2, Q3.4
- new net +5V_HEATER: J5.1
- new net MPPT/VIN: J3.1
Other:
- sheet Converters ports: added 5V_HEATER; removed none
- sheet MPPT ports: added +12V, VIN; removed I_SENSE, OUT
- moved on the sheet: F1
