File: PDU/VBAT_Monitor.kicad_sch (KiCad schematic)
At the start: 6 parts, among them U2 MCP6002-I/P

Commit message: Last revision
Parts:
- removed U2: MCP6002-I/P, PDIP8_300MC_MCH, symbol Capstone:MCP6002-I_P
- added U4: MCP6001UT-I/OT, SOT-23-5_MC_MCH, symbol Capstone:MCP6001UT-I_OT
Connections:
- net +5V: now also U4.5 (VDD)
- net GND: now also U4.2 (VSS)
- net VBAT_SCALED: now also U4.3 (VIN-), U4.4 (VOUT)
- net VINA+: now also U4.1 (VIN+)
- no-connect marks 1 -> 0
Other:
- moved on the sheet: C11, R16, R17, R30, R31
